File: HDMI to CSI.sch (KiCad schematic (older format))
At the start: 5 parts

Commit message: modified Schematic, Cu layers routed
Parts:
- J2: renamed from J?; symbol Conn_01x19 -> Conn_01x20
- gave numbers to parts that had none: 4
Connections:
- net CAM_CLK: now also J2.8 (Pin_8); no longer J2.5 (Pin_5)
- net CAM_GPIO: now also J2.6 (Pin_6); no longer J2.3 (Pin_3)
- net DSI1_C+: now also J2.14 (Pin_14); no longer J2.12 (Pin_12)
- net DSI1_C-: now also J2.12 (Pin_12); no longer J2.14 (Pin_14)
- net DSI1_D0+: now also J2.5 (Pin_5); no longer J2.9 (Pin_9)
- net DSI1_D0-: now also J2.3 (Pin_3); no longer J2.11 (Pin_11)
- net DSI1_D1+: now also J2.11 (Pin_11); no longer J2.6 (Pin_6)
- net DSI1_D1-: now also J2.9 (Pin_9); no longer J2.8 (Pin_8)
- net GND: now also J2.20 (Pin_20)
Changed lines of the file:
@@
 $EndDescr
 $Comp
-L Conn_01x15 J?
+L Conn_01x15 J1
 U 1 1 5AC9041C
 P 4500 3550
-F 0 "J?" H 4500 4350 50  0000 C CNN
+F 0 "J1" H 4500 4350 50  0000 C CNN
 F 1 "RPI/CAM" V 4650 3500 50  0000 C CNN
 F 2 "Connectors_TE-Connectivity:TE_1-84952-5_1x15_P1.0mm_Horizontal" H 4500 3550 50  0001 C CNN
@@
 $EndComp
 $Comp
-L GND #PWR?
+L GND #PWR01
 U 1 1 5AC9053D
 P 4800 4700
-F 0 "#PWR?" H 4800 4450 50  0001 C CNN
+F 0 "#PWR01" H 4800 4450 50  0001 C CNN
 F 1 "GND" H 4800 4550 50  0000 C CNN
 F 2 "" H 4800 4700 50  0001 C CNN
@@
 Connection ~ 4800 3750
 $Comp
-L Conn_01x19 J?
+L Conn_01x20 J2
 U 1 1 5AC905EA
 P 6300 3650
-F 0 "J?" H 6300 4650 50  0000 C CNN
+F 0 "J2" H 6300 4650 50  0000 C CNN
 F 1 "MicroHDMI" V 6400 3700 50  0000 C CNN
 F 2 "Connectors_HDMI:HDMI_Micro-D_Molex_46765-0x01" H 6300 3650 50  0001 C CNN
@@
 $EndComp
 $Comp
-L GND #PWR?
+L GND #PWR02
 U 1 1 5AC90939
 P 6000 4700
-F 0 "#PWR?" H 6000 4450 50  0001 C CNN
+F 0 "#PWR02" H 6000 4450 50  0001 C CNN
 F 1 "GND" H 6000 4550 50  0000 C CNN
 F 2 "" H 6000 4700 50  0001 C CNN
@@
 	4900 4250 4700 4250
 $Comp
-L C C?
+L C C1
 U 1 1 5AC91378
 P 5050 2100
-F 0 "C?" H 5075 2200 50  0000 L CNN
+F 0 "C1" H 5075 2200 50  0000 L CNN
 F 1 "1uF" H 5075 2000 50  0000 L CNN
 F 2 "Capacitors_SMD:C_0402" H 5088 1950 50  0001 C CNN
@@
 	5050 1850 5050 1950
 $Comp
-L GND #PWR?
+L GND #PWR03
 U 1 1 5AC91411
 P 5050 2300
-F 0 "#PWR?" H 5050 2050 50  0001 C CNN
+F 0 "#PWR03" H 5050 2050 50  0001 C CNN
 F 1 "GND" H 5050 2150 50  0000 C CNN
 F 2 "" H 5050 2300 50  0001 C CNN
@@
 	5050 2250 5050 2300
 $Comp
-L C C?
+L C C2
 U 1 1 5AC9147C
 P 5450 2100
-F 0 "C?" H 5475 2200 50  0000 L CNN
+F 0 "C2" H 5475 2200 50  0000 L CNN
 F 1 "1uF" H 5475 2000 50  0000 L CNN
 F 2 "Capacitors_SMD:C_0402" H 5488 1950 50  0001 C CNN
@@
 	5450 1850 5450 1950
 $Comp
-L GND #PWR?
+L GND #PWR04
 U 1 1 5AC91485
 P 5450 2300
-F 0 "#PWR?" H 5450 2050 50  0001 C CNN
+F 0 "#PWR04" H 5450 2050 50  0001 C CNN
 F 1 "GND" H 5450 2150 50  0000 C CNN
 F 2 "" H 5450 2300 50  0001 C CNN
@@
 	5450 2250 5450 2300
 $Comp
-L C C?
+L C C3
 U 1 1 5AC914D7
 P 5850 2100
-F 0 "C?" H 5875 2200 50  0000 L CNN
+F 0 "C3" H 5875 2200 50  0000 L CNN
 F 1 "1uF" H 5875 2000 50  0000 L CNN
 F 2 "Capacitors_SMD:C_0402" H 5888 1950 50  0001 C CNN
@@
 	5850 1850 5850 1950
 $Comp
-L GND #PWR?
+L GND #PWR05
 U 1 1 5AC914E0
 P 5850 2300
-F 0 "#PWR?" H 5850 2050 50  0001 C CNN
+F 0 "#PWR05" H 5850 2050 50  0001 C CNN
 F 1 "GND" H 5850 2150 50  0000 C CNN
 F 2 "" H 5850 2300 50  0001 C CNN
@@
 Wire Wire Line
 	6100 4050 5900 4050
+Text Label 5900 4050 2    60   ~ 0
+DSI1_C+
 Text Label 5900 3850 2    60   ~ 0
-DSI1_C+
-Text Label 5900 4050 2    60   ~ 0
 DSI1_C-
+Text Label 5900 3750 2    60   ~ 0
+DSI1_D1+
+Wire Wire Line
+	5900 3250 6100 3250
+Text Label 5900 3550 2    60   ~ 0
+DSI1_D1-
+Text Label 5900 3150 2    60   ~ 0
+DSI1_D0+
+Text Label 5900 2950 2    60   ~ 0
+DSI1_D0-
 Text Label 5900 3250 2    60   ~ 0
-DSI1_D1+
-Wire Wire Line
-	5900 3250 6100 3250
+CAM_GPIO
 Text Label 5900 3450 2    60   ~ 0
-DSI1_D1-
-Text Label 5900 3550 2    60   ~ 0
-DSI1_D0+
-Text Label 5900 3750 2    60   ~ 0
-DSI1_D0-
-Text Label 5900 2950 2    60   ~ 0
-CAM_GPIO
-Text Label 5900 3150 2    60   ~ 0
 CAM_CLK
 Text Label 5900 2850 2    60   ~ 0
@@
 Wire Wire Line
 	5900 4150 6100 4150
+Wire Wire Line
+	6100 4650 6000 4650
+Connection ~ 6000 4650
 $EndSCHEMATC
