File: HDMI to CSI.kicad_pcb (KiCad board)
At the start: 2 copper layers, 27.5 x 25 mm, 5 parts, among them J1 RPI/CAM, J2 MicroHDMI

Commit message: Finished Silscreen and added Gerber
Other:
- board size 27.5 x 25 mm -> 25.5 x 25 mm
- board text added: "MicroHDMI to CSI"
- board text added: "designed by Miroslav Lakota"
Changed lines of the file:
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@@
     (links 32)
     (no_connects 0)
-    (area 0 0 0 0)
+    (area 126.924999 87.424999 152.575001 112.575001)
     (thickness 1.6)
-    (drawings 6)
+    (drawings 9)
     (tracks 242)
     (zones 0)
@@
   )
   (setup
-    (last_trace_width 0.2)
+    (last_trace_width 0.127)
     (user_trace_width 0.127)
     (user_trace_width 0.1524)
@@
     (visible_elements 7FFFFFFF)
     (pcbplotparams
-      (layerselection 0x00030_80000001)
+      (layerselection 0x010fc_80000001)
       (usegerberextensions false)
-      (excludeedgelayer true)
-      (linewidth 0.100000)
+      (usegerberattributes true)
+      (excludeedgelayer false)
+      (linewidth 0.150000)
       (plotframeref false)
       (viasonmask false)
       (mode 1)
-      (useauxorigin false)
+      (useauxorigin true)
       (hpglpennumber 1)
       (hpglpenspeed 20)
@@
       (outputformat 1)
       (mirror false)
-      (drillshape 1)
+      (drillshape 0)
       (scaleselection 1)
-      (outputdirectory ""))
+      (outputdirectory GerberHDMItoCSI/))
   )
   (net 0 "")
@@
     (tags "capacitor 0402")
     (attr smd)
-    (fp_text reference C1 (at 0 -1.27 270) (layer F.SilkS)
+    (fp_text reference C1 (at 0.975 -1.125 270) (layer F.SilkS)
       (effects (font (size 1 1) (thickness 0.15)))
     )
@@
     (tags "capacitor 0402")
     (attr smd)
-    (fp_text reference C2 (at 0 -1.27 90) (layer F.SilkS)
+    (fp_text reference C2 (at 0 -1.425 90) (layer F.SilkS)
       (effects (font (size 1 1) (thickness 0.15)))
     )
@@
     (tags "capacitor 0402")
     (attr smd)
-    (fp_text reference C3 (at 0 -1.27 90) (layer F.SilkS)
+    (fp_text reference C3 (at 0.75 -1.725 90) (layer F.SilkS)
       (effects (font (size 1 1) (thickness 0.15)))
     )
@@
     (tags "te fpc 84952")
     (attr smd)
-    (fp_text reference J1 (at 0 -4 270) (layer F.SilkS)
-      (effects (font (size 1 1) (thickness 0.15)))
-    )
-    (fp_text value RPI/CAM (at 0 7.7 270) (layer F.Fab)
+    (fp_text reference J1 (at -7 -4 270) (layer F.SilkS)
+      (effects (font (size 1 1) (thickness 0.15)))
+    )
+    (fp_text value RPI/CAM (at 0 6 270) (layer F.Fab)
       (effects (font (size 1 1) (thickness 0.15)))
     )
@@
     (fp_line (start 11.96 7) (end 11.96 -3.3) (layer F.CrtYd) (width 0.05))
     (fp_line (start 11.96 -3.3) (end -11.96 -3.3) (layer F.CrtYd) (width 0.05))
-    (fp_text user %R (at 0 1 270) (layer F.Fab)
+    (fp_text user %R (at 9.5 6 270) (layer F.Fab)
       (effects (font (size 1 1) (thickness 0.15)))
     )
@@
     (tags "hdmi micro type d right angle smd")
     (attr smd)
-    (fp_text reference J2 (at 0 -6.3 90) (layer F.SilkS)
-      (effects (font (size 1 1) (thickness 0.15)))
-    )
-    (fp_text value MicroHDMI (at 0 3.6 90) (layer F.Fab)
+    (fp_text reference J2 (at 0.5 -6.3 90) (layer F.SilkS)
+      (effects (font (size 1 1) (thickness 0.15)))
+    )
+    (fp_text value MicroHDMI (at 5.5 -4 180) (layer F.Fab)
       (effects (font (size 1 1) (thickness 0.15)))
     )
@@
     )
   )
+  (gr_text "MicroHDMI\nto CSI\n" (at 142 107) (layer F.SilkS)
+    (effects (font (size 0.8 0.8) (thickness 0.2)) (justify left))
+  )
+  (gr_text "designed by\nMiroslav Lakota" (at 140 93.5) (layer F.SilkS)
+    (effects (font (size 0.8 0.8) (thickness 0.2)) (justify left))
+  )
+  (gr_text "  designed by \nMiroslav Lakota\n" (at 139.5 96) (layer B.SilkS)
+    (effects (font (size 1.5 1.5) (thickness 0.3)) (justify mirror))
+  )
   (gr_line (start 152.5 104.5) (end 140 112.5) (layer Edge.Cuts) (width 0.15))
   (gr_line (start 152.5 95.5) (end 152.5 104.5) (layer Edge.Cuts) (width 0.15))
   (gr_line (start 140 87.5) (end 152.5 95.5) (layer Edge.Cuts) (width 0.15))
-  (gr_line (start 125 87.5) (end 140 87.5) (layer Edge.Cuts) (width 0.15))
-  (gr_line (start 125 112.5) (end 140 112.5) (layer Edge.Cuts) (width 0.15))
-  (gr_line (start 125 87.5) (end 125 112.5) (layer Edge.Cuts) (width 0.15))
+  (gr_line (start 127 87.5) (end 140 87.5) (layer Edge.Cuts) (width 0.15))
+  (gr_line (start 127 112.5) (end 140 112.5) (layer Edge.Cuts) (width 0.15))
+  (gr_line (start 127 87.5) (end 127 112.5) (layer Edge.Cuts) (width 0.15))
   (segment (start 140.025 107.475) (end 138.875 107.475) (width 0.254) (layer F.Cu) (net 1))
   (segment (start 138.875 107.475) (end 137.275 107.475) (width 0.254) (layer F.Cu) (net 1))
